File: KiCad/HearingAid_ESP/HearingAid_ESP.kicad_pcb (KiCad board)
At the start: 2 copper layers, 69.2 x 22.1 mm, 63 parts, among them J1 12402012E212A, Q1 PMOS, Q2 FS8205A, U1 AP2112K-3.3, U2 MAX98357A, U3 TP4056, U4 DW01A, U5 MAX98357A, U8 ESP32-S3

Commit message: Updating files
Routing:
- net VDD_ESP: track 86.2 -> 86.8 mm

Commit message: Removed microphone footprint
Parts:
- removed MK1, MK3: INMP441ACEZ-R7, INMP441ACEZ-R7:MIC_INMP441ACEZ-R7
